File: docs/PCB Design/HydroBlock/hydroblock.kicad_pcb (KiCad board)
At the start: 4 copper layers, 75.9 x 105.9 mm, 30 parts, among them J1 Conn_01x05, J2 Conn_01x07, J3 Conn_01x05, J4 Conn_01x05, J5 Conn_01x06, J6 Conn_01x05, J7 Conn_01x05, J8 Raspberry_Pi_2_3, J9 Conn_01x03, U3 W25Q32JVSS

Commit message: Hydroblock PCB Rev 0.2
Parts:
- JP1, JP2, JP4: footprint Jumper:SolderJumper-3_P2.0mm_Open_TrianglePad1.0x1.5mm -> Jumper:SolderJumper-3_P1.3mm_Open_RoundedPad1.0x1.5mm_NumberLabels
- JP3: footprint Jumper:SolderJumper-2_P1.3mm_Open_TrianglePad1.0x1.5mm -> Jumper:SolderJumper-2_P1.3mm_Open_RoundedPad1.0x1.5mm
Connections:
- RTC1 pad 1: +3.3V -> GND
- RTC1 pad 2: SCK1 -> +3.3V
- RTC1 pad 4: GND -> SCK1
- U1 pad 12: +5V -> unconnected-(U1-5v-Pad12)
Routing:
- net U2TX/CE0: track 119.8 -> 123.9 mm
- net SDA1: track 121.9 -> 124.8 mm
- net +5V: track 163.4 -> 165.5 mm
- net SCK1: track 111.7 -> 112.8 mm
- net Net-(J5-Pin_3): track 15.7 -> 15.0 mm
- net SCL6: track 22.6 -> 23.2 mm
Other:
- board text added: "Rev.0.2 06032023DD"
