File: docs/PCB Design/HydroBlock/hydroblock.kicad_sch (KiCad schematic)
At the start: 23 parts, among them J1 Conn_01x05, J2 Conn_01x07, J3 Conn_01x05, J4 Conn_01x05, J5 Conn_01x06, J6 Conn_01x05, J7 Conn_01x05, J8 Raspberry_Pi_2_3, J9 Conn_01x03, U3 W25Q32JVSS

Commit message: Hydroblock PCB Rev 0.2
Connections:
- net +5V: no longer U1.12 (5v)
Changed lines of the file:
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@@
-    (stroke (width 0) (type default))
-  )
-  (wire (pts (xy 196.85 45.72) (xy 196.85 30.48))
     (stroke (width 0) (type default))
   )
@@
   )
   (wire (pts (xy 241.3 124.46) (xy 255.27 124.46))
-    (stroke (width 0) (type default))
-  )
-  (wire (pts (xy 194.31 45.72) (xy 196.85 45.72))
     (stroke (width 0) (type default))
   )
@@
         )
       )
-    )
-  )
-  (symbol (lib_id "power:+5V") (at 196.85 30.48 0) (mirror y) (unit 1)
-    (in_bom yes) (on_board yes) (dnp no)
-    (property "Reference" "#PWR021" (at 196.85 34.29 0)
-      (effects (font (size 1.27 1.27)) hide)
-    )
-    (property "Value" "+5V" (at 196.85 26.67 0)
-      (effects (font (size 1.27 1.27)))
-    )
-    (property "Footprint" "" (at 196.85 30.48 0)
-      (effects (font (size 1.27 1.27)) hide)
-    )
-    (property "Datasheet" "" (at 196.85 30.48 0)
-      (effects (font (size 1.27 1.27)) hide)
-    )
-    (pin "1")
-    (instances
-      (project "hydroblock"
-        (path "/072973dc-7419-47fb-90d2-54b6b9afca16"
-          (reference "#PWR021") (unit 1)
-        )
-      )
