File: docs/PCB Design/HydroB/HydroBall.kicad_pcb (KiCad board)
At the start: 4 copper layers, 75.9 x 105.9 mm, 69 parts, among them IC1 HIH8130-021-001, J1 Conn_01x05, J10 Conn_01x06, J11 Conn_02x05_Top_Bottom, J12 Conn_01x06, J13 Conn_01x06, J14 Conn_02x04_Counter_Clockwise, J2 Conn_01x07, J3 Conn_01x05, J4 Conn_01x05, J5 Conn_01x06, J6 Conn_01x05, J7 Conn_01x05, J8 Raspberry_Pi_2_3, J9 Conn_01x03, Q2 2N7000, U4 INA238AIDGSR, U7 PCA9533DP_02,118, U8 DS3231MZ, U9 LTV-817

Commit message: HydroB rev 0.5
Parts:
- removed J10: Conn_01x06, Connector_JST:JST_XH_B5B-XH-AM_1x05_P2.50mm_Vertical
- removed J12: Conn_01x06, Connector_JST:JST_XH_B3B-XH-AM_1x03_P2.50mm_Vertical
- removed R18: 540R 1/2W, Resistor_SMD:R_1206_3216Metric
- removed R19: 330R, Resistor_SMD:R_1206_3216Metric
- removed R5: 82R, Resistor_SMD:R_1206_3216Metric
- removed TP10: Cap_Sens, TestPoint:TestPoint_Pad_D2.0mm
- removed U9: LTV-817, Package_DIP:DIP-4_W7.62mm
- added logo1: LOGO, cidco:logo cidco, F.Cu at (151.1, 116.5)
- added logo1: LOGO, cidco:logo cidco, B.Cu at (156.0, 116.5)
- BT1: footprint Battery:BatteryHolder_Keystone_3002_1x2032 -> Battery:BatteryHolder_Keystone_1058_1x2032
- Q2: footprint Package_TO_SOT_THT:TO-92_Inline -> Package_TO_SOT_SMD:SOT-23-3
- R3: value 150R -> 1k
- R4: value 82R -> 1k
- moved R4 58.2 mm to (110.0, 49.3), turned to -90 degrees
- moved R3 57.7 mm to (110.9, 45.8), turned to 0 degrees
- moved R20 48.3 mm to (169.8, 66.7), turned to 180 degrees
- moved J13 48.3 mm to (170.8, 61.5)
- moved Q2 45.0 mm to (170.2, 70.3), turned to 180 degrees
- moved R21 39.1 mm to (164.6, 72.1), turned to 180 degrees
- moved D2 18.1 mm to (123.0, 107.8), turned to 90 degrees
- moved C19 16.7 mm to (164.6, 66.9)
- moved C17 16.5 mm to (164.6, 69.6)
- moved J9 15.6 mm to (107.4, 119.7)
- moved C13 15.3 mm to (129.5, 94.3), turned to 90 degrees
- moved C7 11.4 mm to (130.9, 107.6)
- moved IC1 10.6 mm to (159.1, 69.5)
- moved U7 9.61 mm to (148.0, 69.0), turned to 0 degrees
- moved F1 9.56 mm to (107.2, 98.7)
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Connections:
- J11 pad 4: +5V -> Signal
- J11 pad 7: unconnected-(J11-Pin_7-Pad7) -> Red
- J11 pad 8: LedB -> Green
- J11 pad 9: GND -> Pwr_Pulse
- J8 pad 11: CP_S -> unconnected-(J8-GPIO17-Pad11)
- J8 pad 16: unconnected-(J8-GPIO23-Pad16) -> Pwr_Pulse
- R3 pad 1: Net-(J10-Pin_4) -> Pwr_off
- R3 pad 2: Net-(U7-LED0) -> +3.3V
- R4 pad 1: Net-(J10-Pin_3) -> +3.3V
- R4 pad 2: Net-(U7-LED1) -> Pwr_Pulse
- U7 pad 1: Net-(U7-LED0) -> Red
- U7 pad 2: Net-(U7-LED1) -> Green
Routing:
- net LedB: track 66.0 -> 0.00 mm, vias 1 -> 0
- net GND: track 188.5 -> 125.8 mm, vias 0 -> 5
- net Pwr_Pulse: track 0.00 -> 53.9 mm
- net SEN-: track 81.2 -> 27.8 mm
- net Green: track 0.00 -> 49.1 mm, vias 0 -> 1
- net Red: track 0.00 -> 48.1 mm, vias 0 -> 1
- net Net-(BT1-+): track 50.9 -> 7.97 mm
- net SEN+: track 81.7 -> 41.9 mm
- net CP_S: track 34.7 -> 0.00 mm
- net +3.3V: track 80.3 -> 46.8 mm, vias 3 -> 6
- net SCK4: track 197.6 -> 179.8 mm
- net SDA4: track 188.9 -> 175.2 mm
- net Net-(D2-A): track 4.75 -> 17.5 mm
- net Net-(PS1-VIN): track 44.5 -> 33.2 mm
- net Net-(U7-LED0): track 9.90 -> 0.00 mm
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Other:
- board text added: "PN: HB-HAT Rev.05 10022025DD"
- board text removed: "CS"
- board text removed: "LED"
- board text removed: "PN: HB-HAT Rev.0.3 18092024DD"
