File: docs/PCB Design/HydroB/HydroBall.kicad_sch (KiCad schematic)
At the start: 69 parts, among them IC1 HIH8130-021-001, J1 Conn_01x05, J10 Conn_01x06, J11 Conn_02x05_Top_Bottom, J12 Conn_01x06, J13 Conn_01x06, J14 Conn_02x04_Counter_Clockwise, J2 Conn_01x07, J3 Conn_01x05, J4 Conn_01x05, J5 Conn_01x06, J6 Conn_01x05, J7 Conn_01x05, J8 Raspberry_Pi_2_3, J9 Conn_01x03, Q2 2N7000, U4 INA238AIDGSR, U7 PCA9533DP_02,118, U8 DS3231MZ, U9 LTV-817

Commit message: HydroB rev 0.5
Parts:
- removed J10: Conn_01x06, Connector_JST:JST_XH_B5B-XH-AM_1x05_P2.50mm_Vertical, symbol Connector_Generic:Conn_01x05
- removed J12: Conn_01x06, Connector_JST:JST_XH_B3B-XH-AM_1x03_P2.50mm_Vertical, symbol Connector_Generic:Conn_01x03
- removed R18: 540R 1/2W, Resistor_SMD:R_1206_3216Metric, symbol Device:R_US
- removed R19: 330R, Resistor_SMD:R_1206_3216Metric, symbol Device:R_US
- removed R5: 82R, Resistor_SMD:R_1206_3216Metric, symbol Device:R_US
- removed TP10: Cap_Sens, TestPoint:TestPoint_Pad_D2.0mm, symbol Connector:TestPoint
- removed U9: LTV-817, Package_DIP:DIP-4_W7.62mm, symbol Isolator:LTV-817
- BT1: footprint Battery:BatteryHolder_Keystone_3002_1x2032 -> Battery:BatteryHolder_Keystone_1058_1x2032
- Q2: footprint Package_TO_SOT_THT:TO-92_Inline -> Package_TO_SOT_SMD:SOT-23-3
- R3: value 150R -> 1k
- R4: value 82R -> 1k
Connections:
- net LedB is gone; now on net Green: J11.8 (Pin_8)
- net +3.3V: now also R3.2, R4.1
- net +5V: no longer J11.4 (Pin_4)
- net GND: no longer J11.9 (Pin_9)
- net Pwr_off: now also R3.1
- net Red: now reaches U7.1 (LED0)
- net Red: now also J11.7 (Pin_7); no longer R3.2
- net Green: now reaches U7.2 (LED1)
- net Green: no longer R4.2
- net Pwr_Pulse: now reaches J8.16 (GPIO23)
- net Pwr_Pulse: now also J11.9 (Pin_9), R4.2
- net CP_S: no longer names the net of J8.11 (GPIO17)
- new net Signal: J11.4 (Pin_4)
Other:
- note removed: "Capasitive Sensor"
- note removed: "R G B"
