File: docs/PCB Design/HB-PM-Prog/prog.kicad_pcb (KiCad board)
At the start: 2 copper layers, 38.3 x 62.6 mm, 9 parts, among them J1 Conn_01x08_Pin, J11 Conn_02x05_Top_Bottom, J14 Conn_02x04_Counter_Clockwise, J2 Conn_02x05_Odd_Even, J3 Conn_01x04_Pin

Commit message: update the power module programmer interface to be able to power the power module from a usb port if programmed with an atmel ice programmer
Parts:
- removed J3: Conn_01x04_Pin, Connector_PinHeader_2.54mm:PinHeader_1x04_P2.54mm_Horizontal
- removed R1: 4.7k, Resistor_SMD:R_1206_3216Metric_Pad1.30x1.75mm_HandSolder
- added J4: USB_B, Connector_USB:USB_B_Lumberg_2411_02_Horizontal, F.Cu at (129.8, 92.4)
- moved J1 2.17 mm to (129.0, 64.4)
Routing:
- net Signal: track 80.8 -> 54.6 mm
- net GND: track 116.2 -> 136.2 mm
- net Net-(J3-Pin_2): track 3.45 -> 0.00 mm
- net VCC: track 109.4 -> 110.0 mm
Other:
- board text added: "PN: HB-PM-Prog Rev.1.1 27022025DD"
- board text removed: "PN: HB-PM-Prog Rev.1.0 11022025DD"
