File: docs/PCB Design/HB-PM-Prog/prog.kicad_sch (KiCad schematic)
At the start: 8 parts, among them J1 Conn_01x08_Pin, J11 Conn_02x05_Top_Bottom, J14 Conn_02x04_Counter_Clockwise, J2 Conn_02x05_Odd_Even, J3 Conn_01x04_Pin

Commit message: update the power module programmer interface to be able to power the power module from a usb port if programmed with an atmel ice programmer
Parts:
- removed J3: Conn_01x04_Pin, Connector_PinHeader_2.54mm:PinHeader_1x04_P2.54mm_Horizontal, symbol Connector:Conn_01x04_Pin
- removed R1: 4.7k, Resistor_SMD:R_1206_3216Metric_Pad1.30x1.75mm_HandSolder, symbol Device:R
- added J4: USB_B, Connector_USB:USB_B_Lumberg_2411_02_Horizontal, symbol Connector:USB_B
Connections:
- net +5V: now also J4.1 (VBUS)
- net GND: now also J4.4 (GND), J4.5 (Shield)
